File: eaglecad/rev1/ArduinoInterface_v2.1.sch (EAGLE design)
At the start: 49 parts, among them IC1 74LS00N, IC10 74LS241N, IC11 74LS20N, IC3 74LS30N, IC5 74S74N, IC6 74LS139N, IC7 74LS155N, IC8 74LS241N, IC9 7805TV, J1 Connector, J2 TEENSY_CONN, J3 GLUE_CONN

Commit message: updating schematics
Parts:
- removed C3, C8: .1uf, adafruit:C-US025-025X050
- removed H5, H6, H7, H8: STANDOFF_ELECTRICAL, SparkFun-Hardware:STANDOFF_ELECTRICAL
- removed IC11: 74LS20N, 74xx-us:74LS20N
- removed IC6: 74LS139N, 74xx-us:74LS139N
- removed IC7: 74LS155N, 74xx-us:74LS155N
- removed IC8: 74LS241N, 74xx-us:74LS241N
- removed J2: TEENSY_CONN, SparkFun-Connectors:CONN_13X22X13
- removed J3: GLUE_CONN, SparkFun-Connectors:CONN_13X22X13
- removed R7: 4.7k, resistor:R-US_0204/2V
- added IC2: 74LS373N, 74xx-us:74LS373N
- added IC4: 74LS245N, 74xx-us:74LS245N
- IC10: value 74LS241N -> 74LS04N; device 74xx-us:74LS241N -> 74xx-us:74LS04N
Connections:
- net 37E0RD_LV_ renamed WR_LV
- net 37E0WR_LV_ renamed WR_LV_
- net 37E4WR_LV_ renamed INTERRUPT_LV
- net 37ECRD_LV_ renamed RD_LV_
- net 9V renamed N$12
- net 9V_TO_SW renamed N$22
- net INTERUPT_TO_TRS80_LV_ renamed A2_LV
- removed net 37E0RD_: IC11A.I0, IC7A.1Y0, J3.9
- removed net 37E0RD_HV_SLLC_: B2.HV_TXO_2, J2.9
- removed net 37E0WR_: IC11B.I0, IC7A.2Y0, J3.24
- removed net 37E0WR_LV_SLLC_: B1.HV_RXI_2, J2.24
- removed net 37E4RD_: IC11A.I1, IC7A.1Y1, J3.7
- removed net 37E4RD_HV_SLLC_: B2.HV_RXI_2, J2.7
- removed net 37E4RD_LV_: B2.LV_RXO_2, U$2.11/MOSI
- removed net 37E4WR_: IC11B.I1, IC7A.2Y1, J3.22
- removed net 37E4WR_HV_SLLC_: B1.HV_RXI_1, J2.22
- removed net 37E8RD_: IC11A.I2, IC7A.1Y2, J3.5
- removed net 37E8RD_HV_SLLC_: B2.HV_RXI_1, J2.5
- removed net 37E8RD_LV_: B2.LV_RXO_1, U$2.12/MISO
- removed net 37E8WR_: IC11B.I2, IC7A.2Y2, J3.18
- removed net 37E8WR_HV_SLLC_: B5.HV_TXO_2, J2.18
- removed net 37E8WR_LV_: B5.LV_TXI_2, U$2.33/A14
- removed net 37ECRD_: IC11A.I3, IC7A.1Y3, J3.26
- removed net 37ECRD_HV_SLLC_: B1.HV_TXO_2, J2.26
- removed net 37ECWR_: IC11B.I3, IC7A.2Y3, J3.16
- removed net 37ECWR_HV_SLLC_: B5.HV_RXI_2, J2.16
- removed net 37ECWR_LV_: B5.LV_RXO_2, U$2.34/A15
- removed net 37EXRD: IC11A.O, IC1B.I0, IC1B.I1
- removed net 37EXRD_: IC10B.G, IC1A.I0, IC1B.O, IC8B.G
- removed net 37EXWR: IC11B.O, IC1C.I0, IC1C.I1
- removed net 37EXWR_: IC10A.G, IC1A.I1, IC1C.O, IC8A.G
- removed net 37EX_: IC6B.Y0, IC7A.1G, IC7A.2G
- removed net 37EX_WR_RD: IC1A.O, IC5A.CLK
- removed net 3XXX_: IC6A.Y0, IC6B.G
- removed net A0_HV_SLLC: B5.HV_TXO_1, J2.12
- removed net A14: IC6A.A, U$1.A14
- removed net A1_HV_SLLC: B6.HV_TXO_2, J2.10
- removed net D0_HV: IC10A.Y3, IC10B.A2, J3.25
- removed net D0_HV_SLLC: B3.HV_TXO_2, J2.25
- removed net D1_HV: IC10A.Y2, IC10B.A3, J3.23
- removed net D1_HV_SLLC: B3.HV_RXI_2, J2.23
- removed net D2_HV_SLLC: B3.HV_RXI_1, J2.21
- removed net D3_HV_SLLC: B3.HV_TXO_1, J2.19
- removed net D4_HV_SLLC: B4.HV_TXO_2, J2.17
- removed net D5_HV_SLLC: B4.HV_RXI_2, J2.15
- removed net D6_HV_SLLC: B4.HV_RXI_1, J2.13
- removed net D7_HV_SLLC: B4.HV_TXO_1, J2.11
- removed net FLIPFLOP_CLR_HV_SLLC: B2.HV_TXO_1, J2.3
- removed net FLIPFLOP_PRE_HV: B1.HV_TXO_1, J2.20
- removed net INTERUPT_TO_TRS80_: J3.14, R7.2, U$1.INT*
- removed net INTERUPT_TO_TRS80_HV_SLLC_: B5.HV_RXI_1, J2.14
- removed net NOTHING1_HV_SLLC: B6.HV_RXI_1, J2.6
- removed net NOTHING1_LV: B6.LV_RXO_1, U$2.38/A19
- removed net NOTHING2_HV_SLLC: B6.HV_TXO_1, J2.4
- removed net NOTHING2_LV: B6.LV_TXI_1, U$2.39/A20
- removed net NOTHING3_HV_SLLC: B6.HV_RXI_2, J2.8
- removed net NOTHING3_LV: B6.LV_RXO_2, U$2.30
- removed net RAS_: IC6A.G, U$1.RAS*
- removed net RD: IC1D.O, IC7A.1C
- removed net XX11X111111XXXX: IC3A.O, IC6B.A
- new net A0_AFTER_LATCH: B5.HV_TXO_2, IC2A.1Q
- new net A1_AFTER_LATCH: B5.HV_RXI_2, IC2A.2Q
- new net A2_AFTER_LATCH: B5.HV_RXI_1, IC2A.3Q
- new net A3_AFTER_LATCH: B5.HV_TXO_1, IC2A.4Q
- new net A3_LV: B5.LV_TXI_1, U$2.36/A17
- new net A4: IC2A.5D, U$1.A4
- new net A4_AFTER_LATCH: B6.HV_TXO_2, IC2A.5Q
- new net A4_LV: B6.LV_TXI_2, U$2.37/A18
- new net A5_AFTER_LATCH: B6.HV_RXI_2, IC2A.6Q
- new net A5_LV: B6.LV_RXO_2, U$2.38/A19
- new net A6_AFTER_LATCH: B6.HV_RXI_1, IC2A.7Q
- new net A6_LV: B6.LV_RXO_1, U$2.39/A20
- new net A7_AFTER_LATCH: B6.HV_TXO_1, IC2A.8Q
- new net A7_LV: B6.LV_TXI_1, U$2.30
- new net DATA_BUS_ENABLE_: IC1C.O, IC4A.G
- new net DATA_BUS_ENABLE_HV_FROM_TEENSY: B2.HV_RXI_1, IC1B.I0
- new net DATA_BUS_ENABLE_LV: B2.LV_RXO_1, U$2.24
- new net INTERRUPT: B1.HV_RXI_1, IC1C.I1, IC1D.O, IC2A.ENC, IC5A.CLK, IC5B.CLK
- new net N$13: B3.HV_TXO_2, IC4A.B1
- new net N$2: IC10D.I, U$1.A14
- new net N$24: B3.HV_RXI_2, IC4A.B2
- new net N$26: IC1D.I1, U$1.RAS*
- new net N$3: IC10E.O, IC3A.I0
- new net N$4: IC10D.O, IC3A.I1
- new net N$7: IC1D.I0, IC3A.O
- new net N$8: IC10C.O, IC3A.I2
- new net RDX_OR_WRX_AND_DATA_BUS_ENABLE_FROM_TEENSY: IC10F.O, IC1C.I0
- new net RDX_OR_WRX_AND_DATA_BUS_ENABLE_FROM_TEENSY_: IC10F.I, IC1B.O
- new net READ_OR_WRITE: IC1A.O, IC1B.I1
- new net WR_HV: B2.HV_TXO_2, IC5B.Q
- net A0: now also IC2A.1D; no longer J3.12
- net A0_LV: now also B5.LV_TXI_2, U$2.33/A14; no longer B5.LV_TXI_1, U$2.36/A17
- net A1: now also IC2A.2D; no longer J3.10
- net A11: now also IC10C.I; no longer IC6B.B
- net A12: now also IC3A.I4; no longer IC3A.I6
- net A13: now also IC3A.I3; no longer IC3A.I7
- net A15: now also IC10E.I; no longer IC6A.B
- net A1_LV: now also B5.LV_RXO_2, U$2.34/A15; no longer B6.LV_TXI_2, U$2.37/A18
- net A2: now also IC2A.3D; no longer IC7A.A
- net A3: now also IC2A.4D; no longer IC7A.B
- net A5: now also IC2A.6D; no longer IC3A.I0
- net A6: now also IC2A.7D; no longer IC3A.I1
- net A7: now also IC2A.8D; no longer IC3A.I2
- net A8: now also IC3A.I7; no longer IC3A.I3
- net A9: now also IC3A.I6; no longer IC3A.I4
- net D0: now also IC4A.A1; no longer IC10A.A3, IC10B.Y2
- net D1: now also IC4A.A2; no longer IC10A.A2, IC10B.Y3
- net D2: now also IC4A.A3; no longer IC10A.A4, IC10B.Y1
- net D2_HV: now also B3.HV_RXI_1, IC4A.B3; no longer IC10A.Y4, IC10B.A1, J3.21
- net D3: now also IC4A.A4; no longer IC10A.A1, IC10B.Y4
- net D3_HV: now also B3.HV_TXO_1, IC4A.B4; no longer IC10A.Y1, IC10B.A4, J3.19
- net D4: now also IC4A.A5; no longer IC8A.A1, IC8B.Y4
- net D4_HV: now also B4.HV_TXO_2, IC4A.B5; no longer IC8A.Y1, IC8B.A4, J3.17
- net D5: now also IC4A.A6; no longer IC8A.A4, IC8B.Y1
- net D5_HV: now also B4.HV_RXI_2, IC4A.B6; no longer IC8A.Y4, IC8B.A1, J3.15
- net D6: now also IC4A.A7; no longer IC8A.A3, IC8B.Y2
- net D6_HV: now also B4.HV_RXI_1, IC4A.B7; no longer IC8A.Y3, IC8B.A2, J3.13
- net D7: now also IC4A.A8; no longer IC8A.A2, IC8B.Y3
- net D7_HV: now also B4.HV_TXO_1, IC4A.B8; no longer IC8A.Y2, IC8B.A3, J3.11
- net FLIPFLOP_CLR: now also B2.HV_TXO_1, IC5B.CLR; no longer J3.3
- net FLIPFLOP_PRE: now also B1.HV_TXO_1, IC5B.PRE; no longer J3.20
- net GND: now also IC10A.I, IC10B.I, IC2A.OC, IC2P.GND, IC4P.GND; no longer C3.1, C8.1, H5.P$1, H6.P$1, H7.P$1, H8.P$1, IC11P.GND, IC5B.CLK, IC5B.CLR, IC5B.D, IC5B.PRE, IC6P.GND, IC7P.GND, IC8P.GND, J2.1, J3.1
- net RD_: now also B1.HV_TXO_2, IC1A.I0, IC4A.DIR, IC5B.D; no longer IC1D.I0, IC1D.I1
- net VCC: now also IC2P.VCC, IC4P.VCC; no longer C3.2, C8.2, IC11P.VCC, IC6P.VCC, IC7P.VCC, IC8P.VCC, J2.2, J3.2, R7.1
- net WR_: now also B1.HV_RXI_2, IC1A.I1; no longer IC7A.2C
Other:
- moved on the sheet: B1, B2, B3, B4, B5, B6, C1, C10, C11, C2, C4, C5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
