File: eaglecad/rev1/ArduinoInterface_v3.1.sch (EAGLE design)
At the start: 49 parts, among them IC1 74LS00N, IC10 74LS241N, IC11 74LS20N, IC3 74LS30N, IC5 74S74N, IC6 74LS139N, IC7 74LS155N, IC8 74LS241N, IC9 7805TV, J1 Connector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

Commit message: updating schematics
Parts:
- removed IC10, IC8: 74LS241N, 74xx-us:74LS241N
- added IC2, IC4: 74LS244N, 74xx-us:74LS244N
Connections:
- removed net N$16: R4.1, U$2.20/A6
- removed net N$17: R5.1, U$2.19/A5/SCL
- removed net N$18: R6.1, U$2.18/A4/SDA
- removed net N$9: R3.1, U$2.21/A7
- new net N$3: R6.1, U$2.2
- new net N$4: R5.1, U$2.3/CANTX
- new net N$7: R2.1, U$2.6
- new net N$8: R1.1, U$2.7
- net 37E0RD_LV_: now also U$2.31/A12; no longer U$2.10/CS
- net 37E4RD_LV_: now also U$2.32/A13; no longer U$2.11/MOSI
- net 37E8RD_LV_: now also U$2.30; no longer U$2.12/MISO
- net 37EXRD_: now also IC2B.G, IC4B.G; no longer IC10B.G, IC8B.G
- net 37EXWR_: now also IC2A.G, IC4A.G; no longer IC10A.G, IC8A.G
- net A0_LV: now also U$2.35/A16; no longer U$2.36/A17
- net A1_LV: now also U$2.36/A17; no longer U$2.37/A18
- net D0: now also IC2A.A3, IC2B.Y2; no longer IC10A.A3, IC10B.Y2
- net D0_HV: now also IC2A.Y3, IC2B.A2; no longer IC10A.Y3, IC10B.A2
- net D0_LV: now also U$2.15/A1; no longer U$2.2
- net D1: now also IC2A.A2, IC2B.Y3; no longer IC10A.A2, IC10B.Y3
- net D1_HV: now also IC2A.Y2, IC2B.A3; no longer IC10A.Y2, IC10B.A3
- net D1_LV: now also U$2.22/A8; no longer U$2.3/CANTX
- net D2: now also IC2A.A4, IC2B.Y1; no longer IC10A.A4, IC10B.Y1
- net D2_HV: now also IC2A.Y4, IC2B.A1; no longer IC10A.Y4, IC10B.A1
- net D2_LV: now also U$2.23/A9; no longer U$2.4/CANRX
- net D3: now also IC2A.A1, IC2B.Y4; no longer IC10A.A1, IC10B.Y4
- net D3_HV: now also IC2A.Y1, IC2B.A4; no longer IC10A.Y1, IC10B.A4
- net D3_LV: now also U$2.9/CS; no longer U$2.5
- net D4: now also IC4A.A1, IC4B.Y4; no longer IC8A.A1, IC8B.Y4
- net D4_HV: now also IC4A.Y1, IC4B.A4; no longer IC8A.Y1, IC8B.A4
- net D4_LV: now also U$2.10/CS; no longer U$2.6
- net D5: now also IC4A.A4, IC4B.Y1; no longer IC8A.A4, IC8B.Y1
- net D5_HV: now also IC4A.Y4, IC4B.A1; no longer IC8A.Y4, IC8B.A1
- net D5_LV: now also U$2.13/SCK; no longer U$2.7
- net D6: now also IC4A.A3, IC4B.Y2; no longer IC8A.A3, IC8B.Y2
- net D6_HV: now also IC4A.Y3, IC4B.A2; no longer IC8A.Y3, IC8B.A2
- net D6_LV: now also U$2.11/MOSI; no longer U$2.8
- net D7: now also IC4A.A2, IC4B.Y3; no longer IC8A.A2, IC8B.Y3
- net D7_HV: now also IC4A.Y2, IC4B.A3; no longer IC8A.Y2, IC8B.A3
- net D7_LV: now also U$2.12/MISO; no longer U$2.9/CS
- net GND: now also IC2P.GND, IC4P.GND; no longer IC10P.GND, IC8P.GND
- net INTERUPT_TO_TRS80_LV_: now also U$2.8; no longer U$2.35/A16
- net N$5: now also R4.1, U$2.4/CANRX; no longer R1.1, U$2.23/A9
- net N$6: now also R3.1, U$2.5; no longer R2.1, U$2.22/A8
- net NOTHING3_LV: now also U$2.37/A18; no longer U$2.30
- net VCC: now also IC2P.VCC, IC4P.VCC; no longer IC10P.VCC, IC8P.VCC
Other:
- moved on the sheet: B1, B2, B5, B6, C1, C10, C11, C2, C3, C4, C5, C6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
