File: eaglecad/rev1/ArduinoInterface_v3.brd (EAGLE design)
At the start: 141.9 x 73.3 mm, 49 parts, among them IC1 74LS00N, IC10 74LS241N, IC11 74LS20N, IC3 74LS30N, IC5 74S74N, IC6 74LS139N, IC7 74LS155N, IC8 74LS241N, IC9 7805TV, J1 Connector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

Commit message: updating schematics
Connections:
- net N$12 renamed 9V
- net N$22 renamed 9V_TO_SW
- net N$4 renamed A8
Routing:
- net 9V: track 66.2 -> 89.0 mm, vias 0 -> 2
- net A9: track 49.3 -> 66.8 mm, vias 2 -> 3
- net D5_HV: track 38.9 -> 49.6 mm, vias 1 -> 3
- net VCC: track 0.00 -> 6.86 mm
- net 37E8WR_: track 107.3 -> 113.2 mm, vias 3 -> 5
- net NOTHING2_HV_SLLC: track 84.3 -> 90.1 mm
- net 37E8WR_HV_SLLC_: track 107.0 -> 111.3 mm, vias 4 -> 8
- net FLIPFLOP_PRE_HV: track 52.4 -> 56.4 mm
- net D1: track 69.6 -> 73.5 mm
- net WR_: track 121.2 -> 124.9 mm, vias 1 -> 3
- net 37E4WR_: track 132.7 -> 136.3 mm, vias 2 -> 6
- net 37E4WR_HV_SLLC_: track 53.3 -> 56.7 mm
- net A15: track 84.2 -> 80.9 mm, vias 0 -> 2
- net A2: track 83.2 -> 86.4 mm
- net N$18: track 43.5 -> 46.7 mm, vias 0 -> 2
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Other:
- board size 141.9 x 73.3 mm -> 141.9 x 73.6 mm

Commit message: updated schematic to fix 74LS241/74LS244 mixup
Parts:
- IC2, IC4: value 74LS241N -> 74LS244N
- renumbered IC10 to IC2, IC8 to IC4
Routing:
- net D2_HV: track 46.5 -> 47.7 mm
- net D3: track 45.9 -> 46.9 mm

Commit message: updating schematics
Parts:
- IC10, IC8: value 74LS244N -> 74LS241N
- renumbered IC2 to IC10, IC4 to IC8
Routing:
- net D2_HV: track 47.7 -> 46.5 mm
- net D3: track 46.9 -> 45.9 mm
