File: eaglecad/rev1/ArduinoInterface_v4.brd (EAGLE design)
At the start: 141.9 x 73.6 mm, 49 parts, among them IC1 74LS00N, IC11 74LS20N, IC2 74LS373N, IC3 74LS30N, IC4 74LS244N, IC5 74S74N, IC6 74LS139N, IC7 74LS155N, IC9 7805TV, J1 Connector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

Commit message: updates to v4 schematic
Parts:
- moved C6 76.5 mm to (70.8, 23.8), turned to 90 degrees
- moved R6 64.8 mm to (124.1, 67.9)
- moved R5 64.2 mm to (124.1, 69.8)
- moved R4 63.5 mm to (124.1, 71.8)
- moved RGB_LED1 63.5 mm to (130.2, 4.76), turned to 270 degrees
- moved RGB_LED2 61.3 mm to (130.2, 69.5)
- moved R3 60.4 mm to (126.4, 3.81), turned to 270 degrees
- moved C11 59.6 mm to (81.0, 70.5), turned to 0 degrees
- moved R1 59.3 mm to (129.9, 10.2)
- moved R2 57.9 mm to (128.0, 8.26), turned to 0 degrees
- moved B5 41.6 mm to (97.8, 42.5), turned to 180 degrees
- moved B2 37.4 mm to (133.0, 37.5)
- moved B4 18.7 mm to (97.8, 26.4)
- moved B6 16.5 mm to (133.0, 19.7)
- moved C10 7.65 mm to (81.3, 9.53)
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Connections:
- removed net N$16: R4.1, U$2.20/A6
- removed net N$17: R5.1, U$2.19/A5/SCL
- removed net N$18: R6.1, U$2.18/A4/SDA
- removed net N$9: R3.1, U$2.21/A7
- new net N$3: R6.1, U$2.2
- new net N$4: R5.1, U$2.3/CANTX
- new net N$7: R2.1, U$2.6
- new net N$8: R1.1, U$2.7
- net 37E0RD_LV_: now also U$2.31/A12; no longer U$2.10/CS
- net 37E4RD_LV_: now also U$2.32/A13; no longer U$2.11/MOSI
- net 37E8RD_LV_: now also U$2.30; no longer U$2.12/MISO
- net A0_LV: now also U$2.35/A16; no longer U$2.36/A17
- net A1_LV: now also U$2.36/A17; no longer U$2.37/A18
- net D0_LV: now also U$2.15/A1; no longer U$2.2
- net D1_LV: now also U$2.22/A8; no longer U$2.3/CANTX
- net D2_LV: now also U$2.23/A9; no longer U$2.4/CANRX
- net D3_LV: now also U$2.9/CS; no longer U$2.5
- net D4_LV: now also U$2.10/CS; no longer U$2.6
- net D5_LV: now also U$2.13/SCK; no longer U$2.7
- net D6_LV: now also U$2.11/MOSI; no longer U$2.8
- net D7_LV: now also U$2.12/MISO; no longer U$2.9/CS
- net INTERUPT_TO_TRS80_LV_: now also U$2.8; no longer U$2.35/A16
- net N$5: now also R4.1, U$2.4/CANRX; no longer R1.1, U$2.23/A9
- net N$6: now also R3.1, U$2.5; no longer R2.1, U$2.22/A8
- net NOTHING3_LV: now also U$2.37/A18; no longer U$2.30
Routing:
- net 37E0RD_HV_SLLC_: track 5.92 -> 86.9 mm, vias 0 -> 5
- net 37ECWR_HV_SLLC_: track 145.1 -> 64.3 mm
- net 37E8RD_HV_SLLC_: track 8.15 -> 88.1 mm, vias 0 -> 2
- net 37E4RD_HV_SLLC_: track 5.76 -> 83.9 mm, vias 0 -> 5
- net 37E4RD_LV_: track 4.63 -> 66.0 mm, vias 0 -> 1
- net 37E0RD_LV_: track 4.68 -> 65.8 mm, vias 0 -> 1
- net 37E8WR_HV_SLLC_: track 111.3 -> 53.6 mm, vias 8 -> 4
- net N$7: track 0.00 -> 51.9 mm, vias 0 -> 1
- net NOTHING1_HV_SLLC: track 78.2 -> 127.5 mm, vias 2 -> 5
- net N$16: track 48.7 -> 0.00 mm, vias 2 -> 0
- net INTERUPT_TO_TRS80_HV_SLLC_: track 101.9 -> 54.9 mm, vias 3 -> 4
- net N$18: track 46.7 -> 0.00 mm, vias 2 -> 0
- net N$6: track 16.2 -> 62.7 mm, vias 0 -> 3
- net N$8: track 0.00 -> 46.4 mm, vias 0 -> 1
- net A1_HV_SLLC: track 84.6 -> 130.9 mm, vias 6 -> 3
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
Commit message: update for v3.1 of schematic
Routing:
- net 37EXWR_OUTPUT_ENABLE_: track 50.2 -> 61.2 mm
- net VCC/2: track 106.9 -> 110.3 mm
- net D3_LV: track 14.5 -> 17.6 mm
- net D6_HV: track 69.4 -> 66.6 mm
- net N$5: track 29.2 -> 32.1 mm
- net A1_HV_SLLC: track 130.9 -> 133.5 mm
- net 37E8WR_HV_SLLC_: track 53.6 -> 51.3 mm
- net N$3: track 19.1 -> 21.0 mm
- net D7: track 95.1 -> 97.0 mm
- net D4: track 113.2 -> 114.7 mm
- net FLIPFLOP_PRE: track 67.1 -> 68.5 mm, vias 1 -> 3
- net D2: track 116.2 -> 114.9 mm
- net A2: track 93.2 -> 94.4 mm
- net D0_HV: track 37.3 -> 38.6 mm
- net A7: track 87.8 -> 86.5 mm
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